File: MacroBoard_16keys/MacroBoard_16keys.kicad_pcb (KiCad board)
At the start: 2 copper layers, 20 parts, among them SW1 SW_DIP_x01, SW10 SW_DIP_x01, SW11 SW_DIP_x01, SW12 SW_DIP_x01, SW13 SW_DIP_x01, SW14 SW_DIP_x01, SW15 SW_DIP_x01, SW16 SW_DIP_x01, SW2 SW_DIP_x01, SW3 SW_DIP_x01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

Commit message: Added 3D-model Added Gerber files Added code
Parts:
- removed SW13, SW9: SW_DIP_x01, Button_Switch_Keyboard:SW_Cherry_MX_1.00u_PCB
- added REF**: MountingHole_2.2mm_M2, MountingHole:MountingHole_2.2mm_M2, F.Cu at (166.9, 59.2)
- added REF**: MountingHole_2.2mm_M2, MountingHole:MountingHole_2.2mm_M2, F.Cu at (112.9, 59.1)
- added U1: ProMicro, Arduino Micro Pro:ProMicro, B.Cu at (139.6, 55.8)
- D1, D2, D3, D4: value LED -> LED_RGB; footprint LED_SMD:LED_0201_0603Metric_Pad0.64x0.40mm_HandSolder -> LED_SMD:LED_RGB_5050-6; moved to B.Cu
- SW1, SW5: value SW_DIP_x01 -> RotaryEncoder_Switch; footprint Button_Switch_Keyboard:SW_Cherry_MX_1.00u_PCB -> Rotary_Encoder:RotaryEncoder_Alps_EC11E-Switch_Vertical_H20mm
- moved D2 94.4 mm to (160.1, 103.1), turned to 180 degrees
- moved D1 91.4 mm to (166.9, 47.2), turned to 180 degrees
- moved SW4 72.2 mm to (107.1, 118.7), turned to 180 degrees
- moved SW1 64.7 mm to (105.3, 44.6)
- moved SW15 62.8 mm to (167.1, 98.7), turned to 180 degrees
- moved D3 59.2 mm to (120.1, 103.1), turned to 180 degrees
- moved SW12 56.6 mm to (147.1, 118.7), turned to 180 degrees
- moved SW10 52.5 mm to (147.1, 78.7), turned to 180 degrees
- moved SW3 46.6 mm to (107.1, 98.7), turned to 180 degrees
- moved SW16 45.9 mm to (167.1, 118.7), turned to 180 degrees
- moved D4 40.4 mm to (112.9, 47.1), turned to 180 degrees
- moved SW14 30.8 mm to (167.1, 78.7), turned to 180 degrees
- moved SW8 27.5 mm to (127.1, 118.7), turned to 180 degrees
- moved SW2 27.4 mm to (107.1, 78.7), turned to 180 degrees
- moved SW7 27.4 mm to (127.1, 98.7), turned to 180 degrees
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Connections:
- D1 pad 1: unconnected-(D1-Pad1) -> GND
- D1 pad 2: unconnected-(D1-Pad2) -> GND
- D2 pad 1: unconnected-(D2-Pad1) -> GND
- D2 pad 2: unconnected-(D2-Pad2) -> GND
- D3 pad 1: unconnected-(D3-Pad1) -> GND
- D3 pad 2: unconnected-(D3-Pad2) -> GND
- D4 pad 1: unconnected-(D4-Pad1) -> GND
- D4 pad 2: unconnected-(D4-Pad2) -> GND
- SW10 pad 1: unconnected-(SW10-Pad1) -> Net-(SW10-Pad1)
- SW10 pad 2: unconnected-(SW10-Pad2) -> Net-(SW10-Pad2)
- SW11 pad 1: unconnected-(SW11-Pad1) -> Net-(SW11-Pad1)
- SW11 pad 2: unconnected-(SW11-Pad2) -> Net-(SW10-Pad2)
- SW12 pad 1: unconnected-(SW12-Pad1) -> Net-(SW12-Pad1)
- SW12 pad 2: unconnected-(SW12-Pad2) -> Net-(SW10-Pad2)
- SW14 pad 1: unconnected-(SW14-Pad1) -> Net-(SW10-Pad1)
- SW14 pad 2: unconnected-(SW14-Pad2) -> Net-(SW14-Pad2)
- SW15 pad 1: unconnected-(SW15-Pad1) -> Net-(SW11-Pad1)
- SW15 pad 2: unconnected-(SW15-Pad2) -> Net-(SW14-Pad2)
- SW16 pad 1: unconnected-(SW16-Pad1) -> Net-(SW12-Pad1)
- SW16 pad 2: unconnected-(SW16-Pad2) -> Net-(SW14-Pad2)
- SW2 pad 1: unconnected-(SW2-Pad1) -> Net-(SW10-Pad1)
- SW2 pad 2: unconnected-(SW2-Pad2) -> Net-(SW2-Pad2)
- SW3 pad 1: unconnected-(SW3-Pad1) -> Net-(SW11-Pad1)
- SW3 pad 2: unconnected-(SW3-Pad2) -> Net-(SW2-Pad2)
- SW4 pad 1: unconnected-(SW4-Pad1) -> Net-(SW12-Pad1)
- SW4 pad 2: unconnected-(SW4-Pad2) -> Net-(SW2-Pad2)
- SW6 pad 1: unconnected-(SW6-Pad1) -> Net-(SW10-Pad1)
- SW6 pad 2: unconnected-(SW6-Pad2) -> Net-(SW6-Pad2)
- SW7 pad 1: unconnected-(SW7-Pad1) -> Net-(SW11-Pad1)
- SW7 pad 2: unconnected-(SW7-Pad2) -> Net-(SW6-Pad2)
- SW8 pad 1: unconnected-(SW8-Pad1) -> Net-(SW12-Pad1)
- SW8 pad 2: unconnected-(SW8-Pad2) -> Net-(SW6-Pad2)
Routing:
- net GND: track 0.00 -> 225.4 mm, vias 0 -> 1
- net Net-(D1-Pad5): track 0.00 -> 207.9 mm, vias 0 -> 1
- net Net-(D1-Pad4): track 0.00 -> 202.4 mm, vias 0 -> 3
- net Net-(D1-Pad6): track 0.00 -> 195.9 mm
- net Net-(SW12-Pad1): track 0.00 -> 121.4 mm
- net Net-(SW11-Pad1): track 0.00 -> 98.9 mm, vias 0 -> 2
- net Net-(SW2-Pad2): track 0.00 -> 95.8 mm, vias 0 -> 4
- net Net-(SW14-Pad2): track 0.00 -> 82.3 mm, vias 0 -> 2
- net Net-(SW6-Pad2): track 0.00 -> 73.0 mm, vias 0 -> 4
- net Net-(SW10-Pad1): track 0.00 -> 72.7 mm, vias 0 -> 2
- net Net-(SW10-Pad2): track 0.00 -> 68.2 mm, vias 0 -> 4
- net Net-(SW5-PadS1): track 0.00 -> 54.7 mm
- net Net-(SW1-PadA): track 0.00 -> 40.1 mm
- net Net-(SW1-PadS1): track 0.00 -> 39.3 mm, vias 0 -> 1
- net Net-(SW5-PadB): track 0.00 -> 38.5 mm
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Other:
- board outline added: 79.9 x 85.9 mm
